Commit message: + Collision Checking Working! Need to check mesh collisions still

File: urdf/g1_29dof_lock_waist.urdf (robot description, URDF)
Before this commit: robot g1_29dof_lock_waist, 40 links, 39 joints
Links:
- link left_rubber_hand: geometry collision box size=0.20 0.07 0.10; visual mesh filename=package://fcl_self_collision_checker/urdf/meshes/left_rubbe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
- link right_rubber_hand: geometry collision box size=0.20 0.07 0.10; visual mesh filename=package://fcl_self_collision_checker/urdf/meshes/right_rubb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

Commit message: + Added 1cm safety margin to robot meshes

File: urdf/g1_29dof_lock_waist.urdf (robot description, URDF)
Before this commit: robot g1_29dof_lock_waist, 40 links, 39 joints
Links:
- link head_link: geometry collision mesh filename=package://fcl_self_collision_checker/urdf/meshes/head_link_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; visual mesh filename=package://fcl_self_collision_checker/urdf/meshes/head_link.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
- link left_rubber_hand: geometry collision mesh filename=package://fcl_self_collision_checker/urdf/meshes/left_rubbe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; visual mesh filename=package://fcl_self_collision_checker/urdf/meshes/left_rubbe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
- link logo_link: geometry collision mesh filename=package://fcl_self_collision_checker/urdf/meshes/logo_link_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; visual mesh filename=package://fcl_self_collision_checker/urdf/meshes/logo_link.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
- link right_rubber_hand: geometry collision mesh filename=package://fcl_self_collision_checker/urdf/meshes/right_rubb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; visual mesh filename=package://fcl_self_collision_checker/urdf/meshes/right_rubb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
